File: PCB.kicad_pcb (KiCad board)
At the start: 2 copper layers, 45 x 45 mm, 8 parts, among them SW1 SW_Push, SW2 SW_Push

Commit message: Update PCB.kicad_pcb
Added GitHub link
Other:
- board text added: "github.com/H-Pulis/ESP32-S3_GPIO-AMP"
Changed lines of the file:
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@@
 		)
 		(fp_text user "${REFERENCE}"
-			(at 0 10.16 360)
+			(at 0 10.16 0)
 			(layer "F.Fab")
 			(effects
@@
 		(layer "Edge.Cuts")
 	)
+	(gr_text "github.com/H-Pulis/ESP32-S3_GPIO-AMP"
+		(at 176.5 124.25 0)
+		(layer "B.SilkS")
+		(effects
+			(font
+				(size 1 1)
+				(thickness 0.1)
+				(bold yes)
+			)
+			(justify left bottom mirror)
+		)
+	)
 	(gr_text "MCU1"
